Commit message: modifiche

File: urdf/arm.urdf.xacro (robot description, xacro)
@@ -16,5 +16,5 @@
     <!-- Corpo del robot, plugin Gazebo e ros2_control -->
     <xacro:include filename="armando_body.urdf.xacro"/>
-    <!-- Camera end-effector - commentare per escludere dal modello
-    <xacro:include filename="armando_camera.urdf.xacro"/>-->
+    <!-- Camera end-effector - commentare per escludere dal modello -->
+    <xacro:include filename="armando_camera.urdf.xacro"/>
 </robot>

File: urdf/armando_body.urdf.xacro (robot description, xacro)
@@ -297,4 +297,8 @@
     </joint>
     <link name="dyn5_r"/>
+    <!-- ==== CRUCIALE: Previene la fusione del link della pinza con gli altri link ==== -->
+    <gazebo reference="wrist_rotate_dyn5">
+        <preserveFixedJoint>true</preserveFixedJoint>
+    </gazebo>
     <joint name="wrist_rotate_dyn5" type="fixed">
         <parent link="dyn5_r"/>
@@ -310,20 +314,45 @@
             <material name="orange"/>
         </visual>
-        <collision>
-            <geometry>
-                <mesh filename="file://${pkg_path}/meshes/the_crawer_base.stl" scale="0.001 0.001 0.001"/>
-            </geometry>
-            <origin rpy="0 0 0" xyz="0 0 0"/>
-        </collision>
-        <inertial>
-            <mass value="0.1"/>
-            <inertia ixx="6.90013881e-05" ixy="0.0" ixz="0.0" iyy="1.24554875e-04" iyz="0.0" izz="1.04295793e-04"/>
-        </inertial>
-    </link>
-    <!-- Le pinze rimangono solo come visualizzazione grafica: link fissi -->
+        <collision name="crawer_base_collision">
+            <geometry>
+                <box size="0.07 0.03 0.01"/>
+            </geometry>
+            <origin rpy="0 0 0" xyz="0 0.02 0"/>
+        </collision>
+        <inertial>
+            <mass value="0.1"/>
+            <inertia ixx="6.90013881e-05" ixy="0.0" ixz="0.0" iyy="1.24554875e-04" iyz="0.0" izz="1.04295793e-04"/>
+        </inertial>
+    </link>
+    <!-- ==== CRUCIALE: Configurazione del Sensore di Contatto ==== -->
+    <gazebo reference="crawer_base">
+        <sensor name="contact_sensor" type="contact">
+            <always_on>true</always_on>
+            <update_rate>50.0</update_rate>
+            <contact>
+                <collision>crawer_base_collision</collision>
+            </contact>
+        </sensor>
+    </gazebo>
+    <joint name="gripper_actuator_joint" type="fixed">
+        <parent link="crawer_base"/>
+        <child link="gripper_actuator_link"/>
+        <origin xyz="0 0 0" rpy="0 0 0"/>
+        <axis xyz="0 0 1"/>
+        <limit effort="50" velocity="1.0" lower="-0.6" upper="0.8"/>
+    </joint>
+    <link name="gripper_actuator_link">
+        <inertial>
+            <mass value="0.001"/>
+            <inertia ixx="1e-6" ixy="0.0" ixz="0.0" iyy="1e-6" iyz="0.0" izz="1e-6"/>
+        </inertial>
+    </link>
     <joint name="crawer_base_crawer_left" type="fixed">
         <parent link="crawer_base"/>
         <child link="crawer_left"/>
         <origin xyz="-0.03 0.015 0.01" rpy="0 -1.57 0"/>
+        <axis xyz="0 0 1"/>
+        <limit effort="50" velocity="0.2" lower="-0.012" upper="0.015"/>
+        <mimic joint="gripper_actuator_joint" multiplier="0.01875" offset="0.0"/>
     </joint>
     <link name="crawer_left">
@@ -335,10 +364,4 @@
             <material name="gray"/>
         </visual>
-        <collision>
-            <geometry>
-                <mesh filename="file://${pkg_path}/meshes/the_crawer.stl" scale="0.001 0.001 0.001"/>
-            </geometry>
-            <origin rpy="0 0 0" xyz="0 0 0"/>
-        </collision>
         <inertial>
             <mass value="0.1"/>
@@ -350,4 +373,7 @@
         <child link="crawer_right"/>
         <origin xyz="0.03 0.015 0.01" rpy="3.1415 -1.57 0"/>
+        <axis xyz="0 0 -1"/>
+        <limit effort="50" velocity="0.2" lower="-0.015" upper="0.012"/>
+        <mimic joint="gripper_actuator_joint" multiplier="-0.01875" offset="0.0"/>
     </joint>
     <link name="crawer_right">
@@ -359,10 +385,4 @@
             <material name="green"/>
         </visual>
-        <collision>
-            <geometry>
-                <mesh filename="file://${pkg_path}/meshes/the_crawer.stl" scale="0.001 0.001 0.001"/>
-            </geometry>
-            <origin rpy="0 0 0" xyz="0 0 0"/>
-        </collision>
         <inertial>
             <mass value="0.1"/>
@@ -372,11 +392,10 @@
     <!-- Frame di montaggio della camera (end-effector) -->
     <joint name="camera_mount_joint" type="fixed">
-        <parent link="crawer_base"/>
+        <parent link="base_link"/>
         <child link="camera_mount"/>
-        <origin xyz="0.0 0.03 0.0" rpy="0 0 0"/>
+        <origin xyz="0.0 0.0 1.0" rpy="1.57079632679 1.57079632679 0"/>
     </joint>
     <link name="camera_mount"/>
     <!-- ===== Plugin Gazebo ===== -->
-    <!-- Gazebo Harmonic integration -->
     <gazebo>
         <plugin filename="gz_ros2_control-system" name="gz_ros2_control::GazeboSimROS2ControlPlugin">
@@ -385,10 +404,46 @@
         </plugin>
     </gazebo>
+    <!-- ==== PLUGIN PER AFFERRARE IL CUBO A ==== -->
     <gazebo>
-        <plugin filename="gz-sim-sensors-system" name="gz::sim::systems::Sensors">
-            <render_engine>ogre2</render_engine>
+        <plugin filename="gz-sim-detachable-joint-system" name="gz::sim::systems::DetachableJoint">
+            <parent_link>crawer_base</parent_link>
+            <child_model>obstacle_box_a</child_model>
+            <child_link>link</child_link>
+            <attach_topic>/gripper/attach_a</attach_topic>
+            <detach_topic>/gripper/detach_a</detach_topic>
+            <suppress_child_warning>true</suppress_child_warning>
         </plugin>
     </gazebo>
-    <!-- ===== ros2_control Hardware Interface (Gazebo Harmonic) ===== -->
+    <!-- ==== PLUGIN PER AFFERRARE IL CUBO B ==== -->
+    <gazebo>
+        <plugin filename="gz-sim-detachable-joint-system" name="gz::sim::systems::DetachableJoint">
+            <parent_link>crawer_base</parent_link>
+            <child_model>obstacle_box_b</child_model>
+            <child_link>link</child_link>
+            <attach_topic>/gripper/attach_b</attach_topic>
+            <detach_topic>/gripper/detach_b</detach_topic>
+            <suppress_child_warning>true</suppress_child_warning>
+        </plugin>
+    </gazebo>
+    <!-- ==== PLUGIN PER AFFERRARE IL CUBO C ==== -->
+    <gazebo>
+        <plugin filename="gz-sim-detachable-joint-system" name="gz::sim::systems::DetachableJoint">
+            <parent_link>crawer_base</parent_link>
+            <child_model>obstacle_box_c</child_model>
+            <child_link>link</child_link>
+            <attach_topic>/gripper/attach_c</attach_topic>
+            <detach_topic>/gripper/detach_c</detach_topic>
+        </plugin>
+    </gazebo>
+        <!-- ==== PLUGIN PER AFFERRARE IL CILINDRO D ==== -->
+    <gazebo>
+        <plugin filename="gz-sim-detachable-joint-system" name="gz::sim::systems::DetachableJoint">
+            <parent_link>crawer_base</parent_link>
+            <child_model>obstacle_box_d</child_model>
+            <child_link>link</child_link>
+            <attach_topic>/gripper/attach_d</attach_topic>
+            <detach_topic>/gripper/detach_d</detach_topic>
+        </plugin>
+    </gazebo>
     <ros2_control name="HardwareInterface_Gazebo" type="system">
         <hardware>

File: urdf/armando_camera.urdf.xacro (robot description, xacro)
@@ -15,5 +15,13 @@
         </visual>
     </link>
-    <!-- Sensore camera Gazebo -->
+    <!-- ==== NUOVO: Frame Ottico per la Computer Vision ==== -->
+    <joint name="camera_optical_joint" type="fixed">
+        <parent link="camera_link"/>
+        <child link="camera_optical_frame"/>
+        <!-- Allinea l'asse X di ROS all'asse Z della profondità ottica (OpenCV) -->
+        <origin xyz="0 0 0" rpy="-1.57079632679 0 -1.57079632679"/>
+    </joint>
+    <link name="camera_optical_frame"/>
+    <!-- ==== Plugin Sensore ==== -->
     <gazebo reference="camera_link">
         <sensor name="camera" type="camera">
@@ -21,16 +29,19 @@
                 <horizontal_fov>1.047</horizontal_fov>
                 <image>
-                    <width>320</width>
-                    <height>240</height>
+                    <width>1920</width>
+                    <height>1080</height>
                 </image>
                 <clip>
                     <near>0.1</near>
-                    <far>100</far>
+                    <far>5</far>
                 </clip>
             </camera>
             <always_on>1</always_on>
             <update_rate>30</update_rate>
+            <!-- Ti consiglio di metterlo a true durante il debug per vedere il cono visivo in Gazebo -->
             <visualize>true</visualize>
             <topic>camera</topic>
+            <!-- CRUCIALE: Gazebo firmerà i messaggi con il frame ottico! -->
+            <gz_frame_id>camera_optical_frame</gz_frame_id>
         </sensor>
     </gazebo>
