Commit message: Initial commit: armando_description package (escluso moveit)

File: urdf/armando_body.urdf.xacro (robot description, xacro)
@@ -38,5 +38,7 @@
         </visual>
         <collision>
-            <geometry><box size="0.07 0.07 0.08"/></geometry>
+            <geometry>
+                <mesh filename="file://${pkg_path}/meshes/base_link.stl" scale="0.001 0.001 0.001"/>
+            </geometry>
             <origin rpy="0 0 0" xyz="0 0 0"/>
         </collision>
@@ -60,5 +62,7 @@
         </visual>
         <collision>
-            <geometry><box size="0.05 0.05 0.02"/></geometry>
+            <geometry>
+                <mesh filename="file://${pkg_path}/meshes/base_turn.stl" scale="0.001 0.001 0.001"/>
+            </geometry>
             <origin rpy="0 0 0" xyz="0 0 0"/>
         </collision>
@@ -83,5 +87,7 @@
         </visual>
         <collision>
-            <geometry><box size="0.05 0.05 0.01"/></geometry>
+            <geometry>
+                <mesh filename="file://${pkg_path}/meshes/base_turn_table_rot.stl" scale="0.001 0.001 0.001"/>
+            </geometry>
             <origin rpy="0 0 0" xyz="0 0 0"/>
         </collision>
@@ -105,5 +111,7 @@
         </visual>
         <collision>
-            <geometry><box size="0.03 0.03 0.03"/></geometry>
+            <geometry>
+                <mesh filename="file://${pkg_path}/meshes/dyn.stl" scale="0.01 0.01 0.01"/>
+            </geometry>
             <origin rpy="0 0 0" xyz="0 0 0"/>
         </collision>
@@ -135,5 +143,7 @@
         </visual>
         <collision>
-            <geometry><box size="0.04 0.05 0.02"/></geometry>
+            <geometry>
+                <mesh filename="file://${pkg_path}/meshes/f4_n_f3.stl" scale="0.001 0.001 0.001"/>
+            </geometry>
             <origin rpy="0 0 0" xyz="0 0 0"/>
         </collision>
@@ -157,5 +167,7 @@
         </visual>
         <collision>
-            <geometry><box size="0.03 0.03 0.03"/></geometry>
+            <geometry>
+                <mesh filename="file://${pkg_path}/meshes/dyn.stl" scale="0.01 0.01 0.01"/>
+            </geometry>
             <origin rpy="0 0 0" xyz="0 0 0"/>
         </collision>
@@ -187,5 +199,7 @@
         </visual>
         <collision>
-            <geometry><box size="0.04 0.05 0.02"/></geometry>
+            <geometry>
+                <mesh filename="file://${pkg_path}/meshes/f4_n_f3.stl" scale="0.001 0.001 0.001"/>
+            </geometry>
             <origin rpy="0 0 0" xyz="0 0 0"/>
         </collision>
@@ -209,5 +223,7 @@
         </visual>
         <collision>
-            <geometry><box size="0.03 0.03 0.03"/></geometry>
+            <geometry>
+                <mesh filename="file://${pkg_path}/meshes/dyn.stl" scale="0.01 0.01 0.01"/>
+            </geometry>
             <origin rpy="0 0 0" xyz="0 0 0"/>
         </collision>
@@ -239,5 +255,7 @@
         </visual>
         <collision>
-            <geometry><box size="0.05 0.02 0.01"/></geometry>
+            <geometry>
+                <mesh filename="file://${pkg_path}/meshes/wrist.stl" scale="0.001 0.001 0.001"/>
+            </geometry>
             <origin rpy="0 0 0" xyz="0 0 0"/>
         </collision>
@@ -261,5 +279,7 @@
         </visual>
         <collision>
-            <geometry><box size="0.03 0.03 0.03"/></geometry>
+            <geometry>
+                <mesh filename="file://${pkg_path}/meshes/dyn.stl" scale="0.01 0.01 0.01"/>
+            </geometry>
             <origin rpy="0 0 0" xyz="0 0 0"/>
         </collision>
@@ -291,32 +311,19 @@
         </visual>
         <collision>
-            <geometry><box size="0.03 0.03 0.02"/></geometry>
-            <origin rpy="0 0 0" xyz="0 0 0"/>
-        </collision>
-        <inertial>
-            <mass value="0.1"/>
-            <inertia ixx="6.90013881e-05" ixy="0.0" ixz="0.0" iyy="1.24554875e-04" iyz="0.0" izz="1.04295793e-04"/>
-        </inertial>
-    </link>
-    <joint name="gripper_actuator_joint" type="revolute">
-        <parent link="crawer_base"/>
-        <child link="gripper_actuator_link"/>
-        <origin xyz="0 0 0" rpy="0 0 0"/>
-        <axis xyz="0 0 1"/>
-        <limit effort="50" velocity="1.0" lower="-0.6" upper="0.8"/>
-    </joint>
-    <link name="gripper_actuator_link">
-        <inertial>
-            <mass value="0.001"/>
-            <inertia ixx="1e-6" ixy="0.0" ixz="0.0" iyy="1e-6" iyz="0.0" izz="1e-6"/>
-        </inertial>
-    </link>
-    <joint name="crawer_base_crawer_left" type="prismatic">
+            <geometry>
+                <mesh filename="file://${pkg_path}/meshes/the_crawer_base.stl" scale="0.001 0.001 0.001"/>
+            </geometry>
+            <origin rpy="0 0 0" xyz="0 0 0"/>
+        </collision>
+        <inertial>
+            <mass value="0.1"/>
+            <inertia ixx="6.90013881e-05" ixy="0.0" ixz="0.0" iyy="1.24554875e-04" iyz="0.0" izz="1.04295793e-04"/>
+        </inertial>
+    </link>
+    <!-- Le pinze rimangono solo come visualizzazione grafica: link fissi -->
+    <joint name="crawer_base_crawer_left" type="fixed">
         <parent link="crawer_base"/>
         <child link="crawer_left"/>
         <origin xyz="-0.03 0.015 0.01" rpy="0 -1.57 0"/>
-        <axis xyz="0 0 1"/>
-        <limit effort="50" velocity="0.2" lower="-0.012" upper="0.015"/>
-        <mimic joint="gripper_actuator_joint" multiplier="0.01875" offset="0.0"/>
     </joint>
     <link name="crawer_left">
@@ -329,19 +336,18 @@
         </visual>
         <collision>
-            <geometry><box size="0.04 0.01 0.01"/></geometry>
-            <origin rpy="0 0 0" xyz="0 0 0"/>
-        </collision>
-        <inertial>
-            <mass value="0.1"/>
-            <inertia ixx="6.90013881e-05" ixy="0.0" ixz="0.0" iyy="1.24554875e-04" iyz="0.0" izz="1.04295793e-04"/>
-        </inertial>
-    </link>
-    <joint name="crawer_base_crawer_right" type="prismatic">
+            <geometry>
+                <mesh filename="file://${pkg_path}/meshes/the_crawer.stl" scale="0.001 0.001 0.001"/>
+            </geometry>
+            <origin rpy="0 0 0" xyz="0 0 0"/>
+        </collision>
+        <inertial>
+            <mass value="0.1"/>
+            <inertia ixx="6.90013881e-05" ixy="0.0" ixz="0.0" iyy="1.24554875e-04" iyz="0.0" izz="1.04295793e-04"/>
+        </inertial>
+    </link>
+    <joint name="crawer_base_crawer_right" type="fixed">
         <parent link="crawer_base"/>
         <child link="crawer_right"/>
         <origin xyz="0.03 0.015 0.01" rpy="3.1415 -1.57 0"/>
-        <axis xyz="0 0 -1"/>
-        <limit effort="50" velocity="0.2" lower="-0.015" upper="0.012"/>
-        <mimic joint="gripper_actuator_joint" multiplier="-0.01875" offset="0.0"/>
     </joint>
     <link name="crawer_right">
@@ -354,5 +360,7 @@
         </visual>
         <collision>
-            <geometry><box size="0.04 0.01 0.01"/></geometry>
+            <geometry>
+                <mesh filename="file://${pkg_path}/meshes/the_crawer.stl" scale="0.001 0.001 0.001"/>
+            </geometry>
             <origin rpy="0 0 0" xyz="0 0 0"/>
         </collision>
@@ -391,5 +399,4 @@
         <xacro:hardware_joint name="j2" initial_pos="0.0"/>
         <xacro:hardware_joint name="j3" initial_pos="0.0"/>
-        <xacro:hardware_joint name="gripper_actuator_joint" initial_pos="0.0"/>
     </ros2_control>
 </robot>

Commit message: changes

File: urdf/armando_body.urdf.xacro (robot description, xacro)
@@ -77,5 +77,5 @@
         <origin xyz="-0.0 0.0155 0.013" rpy="0 0 -1.57"/>
         <axis xyz="0 0 1"/>
-        <limit effort="300" velocity="1.0" lower="-2.57" upper="2.57"/>
+        <limit effort="300" velocity="1.0" lower="-3.14" upper="3.14"/>
     </joint>
     <link name="base_turn_rot">
